File: hardware/rp2350-hdmi-hexpansion.kicad_pcb (KiCad board)
At the start: 4 copper layers, 32 x 36.6 mm, 90 parts, among them J1 Hexpansion-Connector, J2 USB-C, J3 SWD, J4 Qwiic, J5 HDMI-A, SW1 BOOTSEL, SW2 RESET, U1 RP2354A, U10 ZD24C64A (fallback), U11 SN74LVC1G07, U2 TPS2116DRLR, U3 TLV62569DBVR, U4 TPS61023DRLR, U6 TPD4E05U06, U7 TPD4E05U06, U8 USBLC6-2SC6, U9 APS6404L-3SQR-SN, Y1 12MHz

Commit message: hardware: WIP schematic and PCB changes from the PC (unreviewed)
Uncommitted working-tree changes found on the Windows checkout, which
was still at b3a3395: schematic last saved 17/10/26 11:57, PCB last
saved 29/09/26 22:18. Pushed to a branch rather than main because the
schematic diff is large (~12.7k lines ignoring line endings) and part of
it is probably KiCad re-save churn. Line endings normalised CRLF -> LF to
match the repo. Review before merging.

Co-Authored-By: Claude Sonnet 5.5 <noreply@anthropic.com>
Claude-Session: https://claude.ai/code/session_01VMD2iSg4JfioYFvgvVDo7J
Parts:
- moved LED3 154.8 mm to (95.7, 146.8)
- moved C15 80.5 mm to (-62.6, 42.2)
- moved C6 76.6 mm to (-63.5, 23.5)
- moved C7 71.1 mm to (-58.0, 23.5)
- moved C17 70.8 mm to (-53.1, 42.3)
- moved U9 35.0 mm to (165.1, 99.2)
- moved Y1 27.2 mm to (115.0, 66.3)
- moved U8 23.1 mm to (132.4, 133.5)
- moved F1 22.5 mm to (137.9, 113.0)
- moved J2 13.0 mm to (141.2, 127.0)
- moved U7 10.3 mm to (127.0, 98.4)
- moved J5 9.97 mm to (133.1, 100.0)
Connections:
- net /+3V3 renamed +3V3
- net /RGB_DIN_R renamed Net-(LED3-DIN)
- C1 pad 2: /GND -> GND
- C10 pad 2: /GND -> GND
- C11 pad 2: /GND -> GND
- C12 pad 2: /GND -> GND
- C13 pad 2: /GND -> GND
- C14 pad 2: /GND -> GND
- C15 pad 2: /GND -> GND
- C16 pad 2: /GND -> GND
- C17 pad 2: /GND -> GND
- C18 pad 2: /GND -> GND
- C2 pad 2: /GND -> GND
- C20 pad 2: /GND -> GND
- C21 pad 2: /GND -> GND
- C22 pad 2: /GND -> GND
- C23 pad 2: /GND -> GND
- C24 pad 2: /GND -> GND
- C25 pad 2: /GND -> GND
- C26 pad 2: /GND -> GND
- C29 pad 2: /GND -> GND
- C3 pad 2: /GND -> GND
- C32 pad 2: /GND -> GND
- C33 pad 2: /GND -> GND
- C4 pad 2: /GND -> GND
- C5 pad 2: /GND -> GND
- C6 pad 2: /GND -> GND
- C7 pad 2: /GND -> GND
- D1 pad 2: /GND -> GND
- H1 pad 1: /GND -> GND
- H2 pad 1: /GND -> GND
- J1 pad 1: /GND -> GND
- J1 pad 10: /GND -> GND
- J1 pad 11: /GND -> GND
- J1 pad 14: /GND -> GND
- J1 pad 17: /GND -> GND
- J1 pad 20: /GND -> GND
- J1 pad 6: /GND -> GND
- J2 pad 13: /GND -> GND
- J2 pad 14: /GND -> GND
- J2 pad A1B12: /GND -> GND
- J2 pad B1A12: /GND -> GND
- J3 pad 2: /GND -> GND
- J4 pad 1: /GND -> GND
- J5 pad 11: /GND -> GND
- J5 pad 17: /GND -> GND
- J5 pad 2: /GND -> GND
- J5 pad 20: /GND -> GND
- J5 pad 21: /GND -> GND
- J5 pad 22: /GND -> GND
- J5 pad 23: /GND -> GND
- J5 pad 5: /GND -> GND
- J5 pad 8: /GND -> GND
- LED1 pad 2: /GND -> GND
- LED2 pad 2: /GND -> GND
- LED3 pad 1: /GND -> GND
- R13 pad 2: /GND -> GND
- R14 pad 1: /3V3_USB -> /MUX_PR1
- R14 pad 2: /MUX_PR1 -> /3V3_USB
- R15 pad 1: /MUX_PR1 -> GND
- R15 pad 2: /GND -> /MUX_PR1
- R17 pad 2: /GND -> GND
- R18 pad 2: /GND -> GND
- R20 pad 2: /GND -> GND
- R35 pad 2: /GND -> GND
- R8 pad 2: /GND -> GND
- R9 pad 2: /GND -> GND
- SW1 pad 2: /GND -> GND
- SW2 pad 2: /GND -> GND
- TP3 pad 1: /GND -> GND
- U1 pad 47: /GND -> GND
- U1 pad 61: /GND -> GND
- U10 pad 1: /GND -> GND
- U10 pad 2: /GND -> GND
- U10 pad 3: /GND -> GND
- U10 pad 4: /GND -> GND
- U10 pad 7: /GND -> GND
- U11 pad 3: /GND -> GND
- U2 pad 1: /GND -> GND
- U3 pad 2: /GND -> GND
- U4 pad 4: /GND -> GND
- U6 pad 3: /GND -> GND
- U6 pad 8: /GND -> GND
- U7 pad 3: /GND -> GND
- U7 pad 8: /GND -> GND
- U8 pad 2: /GND -> GND
- U9 pad 4: /GND -> GND
- Y1 pad 2: /GND -> GND
- Y1 pad 4: /GND -> GND
Routing:
- net GND: vias 0 -> 2
- net /GND: vias 2 -> 0
- added copper zone on B.Cu, net GND
- added copper zone on F.Cu, net GND
- removed copper zone on B.Cu, net /GND
- removed copper zone on F.Cu, net /GND
