File: hardware/rp2350-hdmi-hexpansion.kicad_sch (KiCad schematic)
At the start: 90 parts, among them J1 HDMI-A, J2 USB-C, J3 SWD, J4 Qwiic, J6 Hexpansion-Connector, SW1 BOOTSEL, SW2 RESET, U1 RP2354A, U10 ZD24C64A (fallback), U11 SN74LVC1G07, U2 TPS2116DRLR, U3 TLV62569DBVR, U4 TPS61023DRLR, U6 TPD4E05U06, U7 TPD4E05U06, U8 USBLC6-2SC6, U9 APS6404L-3SQR-SN, Y1 12MHz

Commit message: hardware: edge connector back to J1 and locked in place, HDMI now J5
- Schematic: hexpansion edge connector is J1 again (same symbol UUID as
  the J1 footprint already on the PCB, so Update PCB keeps its position);
  HDMI Type A socket renumbered J1 -> J5. ERC and netlist re-verified.
- PCB: J1 edge connector footprint locked at x 98.25, y 100 mm, F.Cu, so
  layout work can't move it accidentally. Position confirmed unchanged.
- BOMs regenerated for the new references; HISTORY lists the connector
  numbering.

Co-Authored-By: Claude Opus 5.5 <noreply@anthropic.com>
Parts:
- removed J1: HDMI-A, jlc:HDMI-SMD_19P-P0.50-H-F, symbol jlc:HDMI-001
- added J5: HDMI-A, jlc:HDMI-SMD_19P-P0.50-H-F, symbol jlc:HDMI-001
- renumbered J6 to J1
Connections:
- net GND: now also J5.11 (TMDSClockShield), J5.17 (DDC/CECGround), J5.2 (TMDSData2Shield), J5.20, J5.21, J5.22, J5.23, J5.5 (TMDSData1Shield), J5.8 (TMDSData0Shield)
- net HDMI_CK_N: now also J5.12 (TMDSClock-)
- net HDMI_CK_P: now also J5.10 (TMDSClock+)
- net HDMI_D0_N: now also J5.9 (TMDSData0-)
- net HDMI_D0_P: now also J5.7 (TMDSData0+)
- net HDMI_D1_N: now also J5.6 (TMDSData1-)
- net HDMI_D1_P: now also J5.4 (TMDSData1+)
- net HDMI_D2_N: now also J5.3 (TMDSData2-)
- net HDMI_D2_P: now also J5.1 (TMDSData2+)
- net HDMI_HPD: now also J5.19 (HotPlugDetect)
- net V5_HDMI: now also J5.18 (+5VPower)
Changed lines of the file:
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@@
 		(on_board yes)
 		(dnp no)
-		(property "Reference" "J1"
+		(property "Reference" "J5"
 			(at 325.12 190.5 0)
 			(effects
@@
 			(project "rp2350-hdmi-hexpansion"
 				(path "/fb9bfa6e-c44d-469c-aa90-8ec28bcdf17f"
-					(reference "J1")
+					(reference "J5")
 					(unit 1)
 				)
@@
 		(on_board yes)
 		(dnp no)
-		(property "Reference" "J6"
+		(property "Reference" "J1"
 			(at 312.42 312.42 0)
 			(effects
@@
 			(project "rp2350-hdmi-hexpansion"
 				(path "/fb9bfa6e-c44d-469c-aa90-8ec28bcdf17f"
-					(reference "J6")
+					(reference "J1")
 					(unit 1)
 				)

Commit message: hardware: WIP schematic and PCB changes from the PC (unreviewed)
Uncommitted working-tree changes found on the Windows checkout, which
was still at b3a3395: schematic last saved 17/10/26 11:57, PCB last
saved 29/09/26 22:18. Pushed to a branch rather than main because the
schematic diff is large (~12.7k lines ignoring line endings) and part of
it is probably KiCad re-save churn. Line endings normalised CRLF -> LF to
match the repo. Review before merging.

Co-Authored-By: Claude Sonnet 5.5 <noreply@anthropic.com>
Claude-Session: https://claude.ai/code/session_01VMD2iSg4JfioYFvgvVDo7J
Parts:
- C20, R7: now not fitted
Connections:
- net USB_CONN_DP is gone; now on net USB_CONN_DN: J2.A6 (Dp1), J2.B6 (Dp2), R10.1, U8.1 (I/O1), U8.6 (I/O1)
- net 3V3_USB: now also R14.2; no longer R14.1
- net GND: now also R15.1; no longer R15.2
- net MUX_PR1: now also R14.1, R15.2; no longer R14.2, R15.1
- net RGB_DIN_R: no longer names the net of LED3.2 (DIN), R52.2
Other:
- note added: "EEPROM"
- note added: "NEOPIXEL"
- moved on the sheet: C1, C2, C21, C22, C23, C24, C25, C26, C29, C3, C32, C33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
